File: FPS 100/Reverse Engineer/PDP11IF/PDP11IF/PDP11IF_2.kicad_sch (KiCad schematic)
At the start: 25 parts

Commit message: 2025/7/27
Parts:
- added D1: 74LS02, symbol 74xx:74LS02
- added D2: 74LS22, symbol 74xx:74LS22
Connections:
- net at U3.10 (Pin_10): now also D2.8
- net NC: now reaches U3.11 (Pin_11)
- net NC: now also U3.5 (Pin_5), U3.7 (Pin_7), U3.8 (Pin_8), U3.9 (Pin_9)
- net at U3.6 (Pin_6): now also D1.5, D1.6
